Commit message: update add lidar

File: my_mobile_robot/urdf/robot_core.xacro (robot description, xacro)
@@ -1,18 +1,19 @@
 <?xml version="1.0"?>
-<robot xmlns:xacro="http://www.ros.org/wiki/xacro" >
-    <xacro:include filename="inertial_macros.xacro"/>
+<!-- robot_core.xacro -->
+<robot xmlns:xacro="http://www.ros.org/wiki/xacro">
+    <xacro:include filename="inertial_macros.xacro" />
     <xacro:arg name="mesh_enabled" default="false" />
-    <xacro:arg name="robot_namespace" default="/"/>
+    <xacro:arg name="robot_namespace" default="/" />
     <material name="white">
         <color rgba="1 1 1 1" />
     </material>
     <material name="orange">
-        <color rgba="1 0.3 0.1 1"/>
+        <color rgba="1 0.3 0.1 1" />
     </material>
     <material name="blue">
-        <color rgba="0.2 0.2 1 1"/>
+        <color rgba="0.2 0.2 1 1" />
     </material>
     <material name="black">
-        <color rgba="0 0 0 1"/>
+        <color rgba="0 0 0 1" />
     </material>
     <!-- BASE LINK -->
@@ -21,32 +22,32 @@
     <!-- CHASSIS LINK -->
     <joint name="chassis_joint" type="fixed">
-        <parent link="base_link"/>
-        <child link="chassis"/>
-        <origin xyz="-0.1 0 0"/>
+        <parent link="base_link" />
+        <child link="chassis" />
+        <origin xyz="-0.1 0 0" />
     </joint>
     <link name="chassis">
         <visual>
-            <origin xyz="0.15 0 0.075"/>
-            <geometry>
-                <box size="0.3 0.3 0.15"/>
-            </geometry>
-            <material name="white"/>
-        </visual>
-        <collision>
-            <origin xyz="0.15 0 0.075"/>
-            <geometry>
-                <box size="0.3 0.3 0.15"/>
+            <origin xyz="0.15 0 0.075" />
+            <geometry>
+                <box size="0.3 0.3 0.15" />
+            </geometry>
+            <material name="white" />
+        </visual>
+        <collision>
+            <origin xyz="0.15 0 0.075" />
+            <geometry>
+                <box size="0.3 0.3 0.15" />
             </geometry>
         </collision>
         <xacro:inertial_box mass="0.5" x="0.3" y="0.3" z="0.15">
-            <origin xyz="0.15 0 0.075" rpy="0 0 0"/>
+            <origin xyz="0.15 0 0.075" rpy="0 0 0" />
         </xacro:inertial_box>
     </link>
     <!-- LEFT WHEEL LINK -->
     <joint name="left_wheel" type="continuous">
-        <parent link="base_link"/>
-        <child link="left_wheel_link"/>
+        <parent link="base_link" />
+        <child link="left_wheel_link" />
         <origin xyz="0 0.175 0" rpy="-${pi/2} 0 0" />
-        <axis xyz="0 0 1"/>
+        <axis xyz="0 0 1" />
         <dynamics damping="0.5" friction="100.0" />
     </joint>
@@ -54,15 +55,15 @@
         <visual>
             <geometry>
-                <cylinder radius="0.05" length="0.04"/>
-            </geometry>
-            <material name="blue"/>
-        </visual>
-        <collision>
-            <geometry>
-                <cylinder radius="0.05" length="0.04"/>
+                <cylinder radius="0.05" length="0.04" />
+            </geometry>
+            <material name="blue" />
+        </visual>
+        <collision>
+            <geometry>
+                <cylinder radius="0.05" length="0.04" />
             </geometry>
         </collision>
         <xacro:inertial_cylinder mass="0.1" length="0.04" radius="0.05">
-            <origin xyz="0 0 0" rpy="0 0 0"/>
+            <origin xyz="0 0 0" rpy="0 0 0" />
         </xacro:inertial_cylinder>
     </link>
@@ -78,8 +79,8 @@
     <!-- RIGHT WHEEL LINK -->
     <joint name="right_wheel" type="continuous">
-        <parent link="base_link"/>
-        <child link="right_wheel_link"/>
+        <parent link="base_link" />
+        <child link="right_wheel_link" />
         <origin xyz="0 -0.175 0" rpy="${pi/2} 0 0" />
-        <axis xyz="0 0 -1"/>
+        <axis xyz="0 0 -1" />
         <dynamics damping="0.5" friction="100.0" />
     </joint>
@@ -87,15 +88,15 @@
         <visual>
             <geometry>
-                <cylinder radius="0.05" length="0.04"/>
-            </geometry>
-            <material name="blue"/>
-        </visual>
-        <collision>
-            <geometry>
-                <cylinder radius="0.05" length="0.04"/>
+                <cylinder radius="0.05" length="0.04" />
+            </geometry>
+            <material name="blue" />
+        </visual>
+        <collision>
+            <geometry>
+                <cylinder radius="0.05" length="0.04" />
             </geometry>
         </collision>
         <xacro:inertial_cylinder mass="0.1" length="0.04" radius="0.05">
-            <origin xyz="0 0 0" rpy="0 0 0"/>
+            <origin xyz="0 0 0" rpy="0 0 0" />
         </xacro:inertial_cylinder>
     </link>
@@ -109,46 +110,114 @@
         </joint>
     </transmission>
-    <!--Front CASTER WHEEL LINK -->
-    <!-- <joint name="caster_wheel_joint" type="fixed">
+    <!--Front
+    CASTER WHEEL LINK -->
+    <joint name="caster_wheel_joint" type="fixed">
+        <parent link="chassis" />
+        <child link="caster_wheel" />
+        <origin xyz="0.24 0 0" />
+        <dynamics damping="0.0" friction="0.0" />
+    </joint>
+    <gazebo reference="caster_wheel">
+        <mu1 value="0.0" />
+        <mu2 value="0.0" />
+        <kp value="10000000.0" />
+        <kd value="1.0" />
+        <fdir1 value="1 0 0" />
+        <material>Gazebo/Grey</material>
+        <turnGravityOff>false</turnGravityOff>
+    </gazebo>
+    <gazebo reference="left_wheel">
+        <mu1 value="100.0" />
+        <mu2 value="100.0" />
+        <kp value="10000000.0" />
+        <kd value="1.0" />
+        <fdir1 value="1 0 0" />
+        <material>Gazebo/Grey</material>
+        <turnGravityOff>false</turnGravityOff>
+    </gazebo>
+    <gazebo reference="right_wheel">
+        <mu1 value="100.0" />
+        <mu2 value="100.0" />
+        <kp value="10000000.0" />
+        <kd value="1.0" />
+        <fdir1 value="1 0 0" />
+        <material>Gazebo/Grey</material>
+        <turnGravityOff>false</turnGravityOff>
+    </gazebo>
+    <link name="caster_wheel">
+        <visual>
+            <geometry>
+                <sphere radius="0.05" />
+            </geometry>
+            <material name="black" />
+        </visual>
+        <collision>
+            <geometry>
+                <sphere radius="0.05" />
+            </geometry>
+        </collision>
+        <xacro:inertial_sphere mass="0.1" radius="0.05">
+            <origin xyz="0 0 0" rpy="0 0 0" />
+        </xacro:inertial_sphere>
+    </link>
+    <!-- Add a Sensor Link -->
+    <link name="lidar_link">
+        <visual>
+            <!-- Visual properties of the lidar sensor -->
+            <geometry>
+                <cylinder radius="0.03" length="0.06" /> <!-- Example shape, adjust as needed -->
+            </geometry>
+            <material name="blue" /> <!-- Example material, adjust as needed -->
+        </visual>
+        <collision>
+            <!-- Collision properties of the lidar sensor -->
+            <geometry>
+                <cylinder radius="0.03" length="0.06" /> <!-- Example shape, adjust as needed -->
+            </geometry>
+        </collision>
+        <!-- Define inertial properties if necessary -->
+    </link>
+    <!-- Attach the Sensor to the Robot -->
+    <joint name="lidar_joint" type="fixed">
         <parent link="chassis"/>
-        <child link="caster_wheel"/>
-        <origin xyz="0.24 0 0"/>
-        <dynamics damping="0.0" friction="0.0" />
-    </joint> -->
-    <joint name="caster_wheel_joint" type="continuous">
-        <parent link="chassis"/>
-        <child link="caster_wheel"/>
-        <origin xyz="0.24 0 0"/>
-        <axis xyz="0 1 0"/> <!-- Axis of rotation perpendicular to the wheel -->
-        <dynamics damping="0.0" friction="0.0" />
-    </joint>
-    <link name="caster_wheel">
-        <visual>
-          <geometry>
-            <sphere radius="0.05"/>
-          </geometry>
-          <material name="black"/>
-        </visual>
-        <collision>
-          <geometry>
-            <sphere radius="0.05"/>
-          </geometry>
-          <surface>
-            <friction>
-              <ode>
-                <mu>0.0</mu> <!-- Set friction to zero -->
-                <mu2>0.0</mu2> <!-- Set friction to zero -->
-              </ode>
-            </friction>
-          </surface>
-        </collision>
-        <xacro:inertial_sphere mass="0.1" radius="0.05">
-          <origin xyz="0 0 0" rpy="0 0 0"/>
-        </xacro:inertial_sphere>
-      </link>
+        <child link="lidar_link"/>
+        <origin xyz="0.2 0 0.2" rpy="0 0 0"/>
+    </joint>
+    <gazebo reference="lidar_link">
+        <material>Gazebo/Red</material>
+        <sensor name="lidar" type="ray">
+            <pose> 0 0 0 0 0 0 </pose>
+            <visualize>true</visualize>
+            <update_rate>10</update_rate>
+            <ray>
+                <scan>
+                    <horizontal>
+                        <samples>360</samples>
+                        <min_angle>-3.14</min_angle>
+                        <max_angle>3.14</max_angle>
+                    </horizontal>
+                </scan>
+                <range>
+                    <min>0.3</min>
+                    <max>12</max>
+                </range>
+            </ray>
+            <!-- <plugin name="laser_controller" filename="libgazebo_ros_ray_sensor.so">
+                <ros>
+                    <argument>~/out:=scan</argument>
+                </ros>
+                <output_type>sensor_msgs/LaserScan</output_type>
+                <frame_name>lidar_link</frame_name>
+            </plugin> -->
+            <plugin name="lidar_controller" filename="libgazebo_ros_laser.so">
+                <topicName>/scan</topicName>
+                <frameName>lidar_link</frameName>
+            </plugin>
+        </sensor>
+    </gazebo>
     <gazebo>
         <plugin name="gazebo_ros_control" filename="libgazebo_ros_control.so">
-        <robotNamespace>$(arg robot_namespace)</robotNamespace>
-        <legacyModeNS>true</legacyModeNS>
+            <robotNamespace>$(arg robot_namespace)</robotNamespace>
+            <legacyModeNS>true</legacyModeNS>
         </plugin>
     </gazebo>

Commit message: update navigation amcl_nomap_prior

File: my_mobile_robot/urdf/robot_core.xacro (robot description, xacro)
@@ -3,4 +3,5 @@
 <robot xmlns:xacro="http://www.ros.org/wiki/xacro">
     <xacro:include filename="inertial_macros.xacro" />
+    <xacro:include filename="lidar.xacro" />
     <xacro:arg name="mesh_enabled" default="false" />
     <xacro:arg name="robot_namespace" default="/" />
@@ -161,59 +162,6 @@
         </xacro:inertial_sphere>
     </link>
-    <!-- Add a Sensor Link -->
-    <link name="lidar_link">
-        <visual>
-            <!-- Visual properties of the lidar sensor -->
-            <geometry>
-                <cylinder radius="0.03" length="0.06" /> <!-- Example shape, adjust as needed -->
-            </geometry>
-            <material name="blue" /> <!-- Example material, adjust as needed -->
-        </visual>
-        <collision>
-            <!-- Collision properties of the lidar sensor -->
-            <geometry>
-                <cylinder radius="0.03" length="0.06" /> <!-- Example shape, adjust as needed -->
-            </geometry>
-        </collision>
-        <!-- Define inertial properties if necessary -->
-    </link>
-    <!-- Attach the Sensor to the Robot -->
-    <joint name="lidar_joint" type="fixed">
-        <parent link="chassis"/>
-        <child link="lidar_link"/>
-        <origin xyz="0.2 0 0.2" rpy="0 0 0"/>
-    </joint>
-    <gazebo reference="lidar_link">
-        <material>Gazebo/Red</material>
-        <sensor name="lidar" type="ray">
-            <pose> 0 0 0 0 0 0 </pose>
-            <visualize>true</visualize>
-            <update_rate>10</update_rate>
-            <ray>
-                <scan>
-                    <horizontal>
-                        <samples>360</samples>
-                        <min_angle>-3.14</min_angle>
-                        <max_angle>3.14</max_angle>
-                    </horizontal>
-                </scan>
-                <range>
-                    <min>0.3</min>
-                    <max>12</max>
-                </range>
-            </ray>
-            <!-- <plugin name="laser_controller" filename="libgazebo_ros_ray_sensor.so">
-                <ros>
-                    <argument>~/out:=scan</argument>
-                </ros>
-                <output_type>sensor_msgs/LaserScan</output_type>
-                <frame_name>lidar_link</frame_name>
-            </plugin> -->
-            <plugin name="lidar_controller" filename="libgazebo_ros_laser.so">
-                <topicName>/scan</topicName>
-                <frameName>lidar_link</frameName>
-            </plugin>
-        </sensor>
-    </gazebo>
+    <!-- Sensors -->
+    <xacro:laser parent_link="base_link" />
     <gazebo>
         <plugin name="gazebo_ros_control" filename="libgazebo_ros_control.so">
